File: kicad/Vibra_V1.kicad_pcb (KiCad board)
At the start: 2 copper layers, 48 x 38 mm, 34 parts, among them J2 UART, J3 LIS3DH_2809_ORIGINAL_SOCKET, SW2 CAL, U1 XIAO ESP32S3

Commit message: Retire la bibliothèque externe des empreintes
Parts:
- C10, C5, C6, C8, C9: footprint Vibra_Reviewed:C_0805_2012Metric_Pad1.18x1.45mm_HandSolder -> C_0805_2012Metric_Pad1.18x1.45mm_HandSolder
- D1, D2, D3, D4, D5: footprint Vibra_Reviewed:LED_0805_2012Metric_Pad1.15x1.40mm_HandSolder -> LED_0805_2012Metric_Pad1.15x1.40mm_HandSolder
- H1, H2, H3, H4: footprint Vibra_Reviewed:MountingHole_3.2mm_M3 -> MountingHole_3.2mm_M3
- H5, H6: footprint Vibra_Reviewed:MountingHole_2.5mm -> MountingHole_2.5mm
- J2: footprint Vibra_Reviewed:UART_1x03_2.54mm_Drill1.10 -> UART_1x03_2.54mm_Drill1.10
- J3: footprint Vibra_Reviewed:Socket_1x08_2.54mm_H8.5 -> Socket_1x08_2.54mm_H8.5
- R10, R11, R12, R13, R4, R7, R8, R9: footprint Vibra_Reviewed:R_0805_2012Metric_Pad1.20x1.40mm_HandSolder -> R_0805_2012Metric_Pad1.20x1.40mm_HandSolder
- SW2: footprint Vibra_Reviewed:PTS526SK15SMTR2LFS -> PTS526SK15SMTR2LFS
- TP3, TP4, TP6, TP7, TP8, TP9: footprint Vibra_Reviewed:TestPoint_Pad_D1.5mm -> TestPoint_Pad_D1.5mm
- U1: footprint Vibra_Reviewed:XIAO_ESP32S3_Sockets -> XIAO_ESP32S3_Sockets
Changed lines of the file:
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@@
 		)
 	)
-	(footprint "Vibra_Reviewed:LED_0805_2012Metric_Pad1.15x1.40mm_HandSolder"
+	(footprint "LED_0805_2012Metric_Pad1.15x1.40mm_HandSolder"
 		(layer "F.Cu")
 		(at 138 84.5)
@@
 		)
 	)
-	(footprint "Vibra_Reviewed:TestPoint_Pad_D1.5mm"
+	(footprint "TestPoint_Pad_D1.5mm"
 		(layer "F.Cu")
 		(at 112 76)
@@
 		(embedded_fonts no)
 	)
-	(footprint "Vibra_Reviewed:R_0805_2012Metric_Pad1.20x1.40mm_HandSolder"
+	(footprint "R_0805_2012Metric_Pad1.20x1.40mm_HandSolder"
 		(layer "F.Cu")
 		(at 123 80.5 90)
@@
 		)
 	)
-	(footprint "Vibra_Reviewed:MountingHole_3.2mm_M3"
+	(footprint "MountingHole_3.2mm_M3"
 		(layer "F.Cu")
 		(at 103.5 53.5)
@@
 		(embedded_fonts no)
 	)
-	(footprint "Vibra_Reviewed:XIAO_ESP32S3_Sockets"
+	(footprint "XIAO_ESP32S3_Sockets"
 		(layer "F.Cu")
 		(at 116.5 61 90)
@@
 		)
 	)
-	(footprint "Vibra_Reviewed:MountingHole_2.5mm"
+	(footprint "MountingHole_2.5mm"
 		(layer "F.Cu")
 		(at 128.76 75.73)
@@
 		(embedded_fonts no)
 	)
-	(footprint "Vibra_Reviewed:TestPoint_Pad_D1.5mm"
+	(footprint "TestPoint_Pad_D1.5mm"
 		(layer "F.Cu")
 		(at 124.5 77)
@@
 		(embedded_fonts no)
 	)
-	(footprint "Vibra_Reviewed:C_0805_2012Metric_Pad1.18x1.45mm_HandSolder"
+	(footprint "C_0805_2012Metric_Pad1.18x1.45mm_HandSolder"
 		(layer "F.Cu")
 		(at 135 53)
@@
 		)
 	)
-	(footprint "Vibra_Reviewed:Socket_1x08_2.54mm_H8.5"
+	(footprint "Socket_1x08_2.54mm_H8.5"
 		(layer "F.Cu")
 		(at 144 77 180)
@@
 		)
 	)
-	(footprint "Vibra_Reviewed:LED_0805_2012Metric_Pad1.15x1.40mm_HandSolder"
+	(footprint "LED_0805_2012Metric_Pad1.15x1.40mm_HandSolder"
 		(layer "F.Cu")
 		(at 118 84.5)
@@
 		)
 	)
-	(footprint "Vibra_Reviewed:LED_0805_2012Metric_Pad1.15x1.40mm_HandSolder"
+	(footprint "LED_0805_2012Metric_Pad1.15x1.40mm_HandSolder"
 		(layer "F.Cu")
 		(at 123 84.5)
@@
 		)
 	)
-	(footprint "Vibra_Reviewed:R_0805_2012Metric_Pad1.20x1.40mm_HandSolder"
+	(footprint "R_0805_2012Metric_Pad1.20x1.40mm_HandSolder"
 		(layer "F.Cu")
 		(at 130 56)
@@
 		)
 	)
-	(footprint "Vibra_Reviewed:R_0805_2012Metric_Pad1.20x1.40mm_HandSolder"
+	(footprint "R_0805_2012Metric_Pad1.20x1.40mm_HandSolder"
 		(layer "F.Cu")
 		(at 115 75.5 90)
@@
 		)
 	)
-	(footprint "Vibra_Reviewed:MountingHole_3.2mm_M3"
+	(footprint "MountingHole_3.2mm_M3"
 		(layer "F.Cu")
 		(at 103.5 84.5)
@@
 		(embedded_fonts no)
 	)
-	(footprint "Vibra_Reviewed:R_0805_2012Metric_Pad1.20x1.40mm_HandSolder"
+	(footprint "R_0805_2012Metric_Pad1.20x1.40mm_HandSolder"
 		(layer "F.Cu")
 		(at 135 56)
@@
 		)
 	)
-	(footprint "Vibra_Reviewed:C_0805_2012Metric_Pad1.18x1.45mm_HandSolder"
+	(footprint "C_0805_2012Metric_Pad1.18x1.45mm_HandSolder"
 		(layer "F.Cu")
 		(at 134 66.5)
@@
 		)
 	)
-	(footprint "Vibra_Reviewed:R_0805_2012Metric_Pad1.20x1.40mm_HandSolder"
+	(footprint "R_0805_2012Metric_Pad1.20x1.40mm_HandSolder"
 		(layer "F.Cu")
 		(at 118 80.5 90)
@@
 		)
 	)
-	(footprint "Vibra_Reviewed:C_0805_2012Metric_Pad1.18x1.45mm_HandSolder"
+	(footprint "C_0805_2012Metric_Pad1.18x1.45mm_HandSolder"
 		(layer "F.Cu")
 		(at 134 70)
@@
 		)
 	)
-	(footprint "Vibra_Reviewed:UART_1x03_2.54mm_Drill1.10"
+	(footprint "UART_1x03_2.54mm_Drill1.10"
 		(layer "F.Cu")
 		(at 103.5 74 90)
@@
 		)
 	)
-	(footprint "Vibra_Reviewed:R_0805_2012Metric_Pad1.20x1.40mm_HandSolder"
+	(footprint "R_0805_2012Metric_Pad1.20x1.40mm_HandSolder"
 		(layer "F.Cu")
 		(at 138 80.5 90)
@@
 		)
 	)
-	(footprint "Vibra_Reviewed:TestPoint_Pad_D1.5mm"
+	(footprint "TestPoint_Pad_D1.5mm"
 		(layer "F.Cu")
 		(at 124.5 73.5)
@@
 		(embedded_fonts no)
 	)
-	(footprint "Vibra_Reviewed:PTS526SK15SMTR2LFS"
+	(footprint "PTS526SK15SMTR2LFS"
 		(layer "F.Cu")
 		(at 111.5 82.5)
@@
 		)
 	)
-	(footprint "Vibra_Reviewed:LED_0805_2012Metric_Pad1.15x1.40mm_HandSolder"
+	(footprint "LED_0805_2012Metric_Pad1.15x1.40mm_HandSolder"
 		(layer "F.Cu")
 		(at 128 84.5)
@@
 		)
 	)
-	(footprint "Vibra_Reviewed:C_0805_2012Metric_Pad1.18x1.45mm_HandSolder"
+	(footprint "C_0805_2012Metric_Pad1.18x1.45mm_HandSolder"
 		(layer "F.Cu")
 		(at 130 53)
@@
 		)
 	)
-	(footprint "Vibra_Reviewed:MountingHole_2.5mm"
+	(footprint "MountingHole_2.5mm"
 		(layer "F.Cu")
 		(at 128.76 60.49)
@@
 		(embedded_fonts no)
 	)
-	(footprint "Vibra_Reviewed:TestPoint_Pad_D1.5mm"
+	(footprint "TestPoint_Pad_D1.5mm"
 		(layer "F.Cu")
 		(at 137 74)
@@
 		(embedded_fonts no)
 	)
-	(footprint "Vibra_Reviewed:R_0805_2012Metric_Pad1.20x1.40mm_HandSolder"
+	(footprint "R_0805_2012Metric_Pad1.20x1.40mm_HandSolder"
 		(layer "F.Cu")
 		(at 133 80.5 90)
@@
 		)
 	)
-	(footprint "Vibra_Reviewed:MountingHole_3.2mm_M3"
+	(footprint "MountingHole_3.2mm_M3"
 		(layer "F.Cu")
 		(at 144.5 84.5)
@@
 		(embedded_fonts no)
 	)
-	(footprint "Vibra_Reviewed:TestPoint_Pad_D1.5mm"
+	(footprint "TestPoint_Pad_D1.5mm"
 		(layer "F.Cu")
 		(at 103.5 65)
@@
 		(embedded_fonts no)
 	)
-	(footprint "Vibra_Reviewed:MountingHole_3.2mm_M3"
+	(footprint "MountingHole_3.2mm_M3"
 		(layer "F.Cu")
 		(at 144.5 53.5)
@@
 		(embedded_fonts no)
 	)
-	(footprint "Vibra_Reviewed:C_0805_2012Metric_Pad1.18x1.45mm_HandSolder"
+	(footprint "C_0805_2012Metric_Pad1.18x1.45mm_HandSolder"
 		(layer "F.Cu")
 		(at 134 63)
@@
 		)
 	)
-	(footprint "Vibra_Reviewed:LED_0805_2012Metric_Pad1.15x1.40mm_HandSolder"
+	(footprint "LED_0805_2012Metric_Pad1.15x1.40mm_HandSolder"
 		(layer "F.Cu")
 		(at 133 84.5)
@@
 		)
 	)
-	(footprint "Vibra_Reviewed:TestPoint_Pad_D1.5mm"
+	(footprint "TestPoint_Pad_D1.5mm"
 		(layer "F.Cu")
 		(at 140 55.5)
@@
 		(embedded_fonts no)
 	)
-	(footprint "Vibra_Reviewed:R_0805_2012Metric_Pad1.20x1.40mm_HandSolder"
+	(footprint "R_0805_2012Metric_Pad1.20x1.40mm_HandSolder"
 		(layer "F.Cu")
 		(at 128 80.5 90)
