File: kicad/Vibra_V1.kicad_sch (KiCad schematic)
At the start: 34 parts, among them J2 UART, J3 LIS3DH_2809_ORIGINAL_SOCKET, SW2 CAL, U1 XIAO ESP32S3

Commit message: Simplifie le rendu et regroupe les fichiers du projet
Other:
- note added: "Souder les 0805 avant les supports. Enficher les modules hors tension. Voir README.md et rendu/composants.csv."
- note removed: "Souder les 0805 avant les supports. Enficher les modules hors tension. Voir GUIDE_MONTAGE.md et la BOM."
Changed lines of the file:
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@@
 		)
 	)
-	(text "Souder les 0805 avant les supports.\nEnficher les modules hors tension.\nVoir GUIDE_MONTAGE.md et la BOM."
+	(text "Souder les 0805 avant les supports.\nEnficher les modules hors tension.\nVoir README.md et rendu/composants.csv."
 		(exclude_from_sim no)
 		(at 13.97 188 0)

Commit message: Retire la bibliothèque externe des empreintes
Parts:
- C10, C5, C6, C8, C9: footprint Vibra_Reviewed:C_0805_2012Metric_Pad1.18x1.45mm_HandSolder -> C_0805_2012Metric_Pad1.18x1.45mm_HandSolder
- D1, D2, D3, D4, D5: footprint Vibra_Reviewed:LED_0805_2012Metric_Pad1.15x1.40mm_HandSolder -> LED_0805_2012Metric_Pad1.15x1.40mm_HandSolder
- H1, H2, H3, H4: footprint Vibra_Reviewed:MountingHole_3.2mm_M3 -> MountingHole_3.2mm_M3
- H5, H6: footprint Vibra_Reviewed:MountingHole_2.5mm -> MountingHole_2.5mm
- J2: footprint Vibra_Reviewed:UART_1x03_2.54mm_Drill1.10 -> UART_1x03_2.54mm_Drill1.10
- J3: footprint Vibra_Reviewed:Socket_1x08_2.54mm_H8.5 -> Socket_1x08_2.54mm_H8.5
- R10, R11, R12, R13, R4, R7, R8, R9: footprint Vibra_Reviewed:R_0805_2012Metric_Pad1.20x1.40mm_HandSolder -> R_0805_2012Metric_Pad1.20x1.40mm_HandSolder
- SW2: footprint Vibra_Reviewed:PTS526SK15SMTR2LFS -> PTS526SK15SMTR2LFS
- TP3, TP4, TP6, TP7, TP8, TP9: footprint Vibra_Reviewed:TestPoint_Pad_D1.5mm -> TestPoint_Pad_D1.5mm
- U1: footprint Vibra_Reviewed:XIAO_ESP32S3_Sockets -> XIAO_ESP32S3_Sockets
Changed lines of the file:
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@@
 			)
 		)
-		(property "Footprint" "Vibra_Reviewed:XIAO_ESP32S3_Sockets"
+		(property "Footprint" "XIAO_ESP32S3_Sockets"
 			(at 113.03 45.72 0)
 			(hide yes)
@@
 			)
 		)
-		(property "Footprint" "Vibra_Reviewed:Socket_1x08_2.54mm_H8.5"
+		(property "Footprint" "Socket_1x08_2.54mm_H8.5"
 			(at 220.98 44.45 0)
 			(hide yes)
@@
 			)
 		)
-		(property "Footprint" "Vibra_Reviewed:C_0805_2012Metric_Pad1.18x1.45mm_HandSolder"
+		(property "Footprint" "C_0805_2012Metric_Pad1.18x1.45mm_HandSolder"
 			(at 156.21 33.02 0)
 			(hide yes)
@@
 			)
 		)
-		(property "Footprint" "Vibra_Reviewed:MountingHole_2.5mm"
+		(property "Footprint" "MountingHole_2.5mm"
 			(at 139.7 187.96 0)
 			(hide yes)
@@
 			)
 		)
-		(property "Footprint" "Vibra_Reviewed:TestPoint_Pad_D1.5mm"
+		(property "Footprint" "TestPoint_Pad_D1.5mm"
 			(at 111.76 153.67 0)
 			(hide yes)
@@
 			)
 		)
-		(property "Footprint" "Vibra_Reviewed:UART_1x03_2.54mm_Drill1.10"
+		(property "Footprint" "UART_1x03_2.54mm_Drill1.10"
 			(at 104.14 81.28 0)
 			(hide yes)
@@
 			)
 		)
-		(property "Footprint" "Vibra_Reviewed:LED_0805_2012Metric_Pad1.15x1.40mm_HandSolder"
+		(property "Footprint" "LED_0805_2012Metric_Pad1.15x1.40mm_HandSolder"
 			(at 208.28 124.46 0)
 			(hide yes)
@@
 			)
 		)
-		(property "Footprint" "Vibra_Reviewed:MountingHole_3.2mm_M3"
+		(property "Footprint" "MountingHole_3.2mm_M3"
 			(at 78.74 175.26 0)
 			(hide yes)
@@
 			)
 		)
-		(property "Footprint" "Vibra_Reviewed:C_0805_2012Metric_Pad1.18x1.45mm_HandSolder"
+		(property "Footprint" "C_0805_2012Metric_Pad1.18x1.45mm_HandSolder"
 			(at 269.24 48.26 0)
 			(hide yes)
@@
 			)
 		)
-		(property "Footprint" "Vibra_Reviewed:R_0805_2012Metric_Pad1.20x1.40mm_HandSolder"
+		(property "Footprint" "R_0805_2012Metric_Pad1.20x1.40mm_HandSolder"
 			(at 251.46 83.82 0)
 			(hide yes)
@@
 			)
 		)
-		(property "Footprint" "Vibra_Reviewed:MountingHole_3.2mm_M3"
+		(property "Footprint" "MountingHole_3.2mm_M3"
 			(at 50.8 175.26 0)
 			(hide yes)
@@
 			)
 		)
-		(property "Footprint" "Vibra_Reviewed:C_0805_2012Metric_Pad1.18x1.45mm_HandSolder"
+		(property "Footprint" "C_0805_2012Metric_Pad1.18x1.45mm_HandSolder"
 			(at 156.21 53.34 0)
 			(hide yes)
@@
 			)
 		)
-		(property "Footprint" "Vibra_Reviewed:C_0805_2012Metric_Pad1.18x1.45mm_HandSolder"
+		(property "Footprint" "C_0805_2012Metric_Pad1.18x1.45mm_HandSolder"
 			(at 269.24 27.94 0)
 			(hide yes)
@@
 			)
 		)
-		(property "Footprint" "Vibra_Reviewed:MountingHole_3.2mm_M3"
+		(property "Footprint" "MountingHole_3.2mm_M3"
 			(at 22.86 175.26 0)
 			(hide yes)
@@
 			)
 		)
-		(property "Footprint" "Vibra_Reviewed:PTS526SK15SMTR2LFS"
+		(property "Footprint" "PTS526SK15SMTR2LFS"
 			(at 38.1 101.6 0)
 			(hide yes)
@@
 			)
 		)
-		(property "Footprint" "Vibra_Reviewed:TestPoint_Pad_D1.5mm"
+		(property "Footprint" "TestPoint_Pad_D1.5mm"
 			(at 154.94 153.67 0)
 			(hide yes)
@@
 			)
 		)
-		(property "Footprint" "Vibra_Reviewed:R_0805_2012Metric_Pad1.20x1.40mm_HandSolder"
+		(property "Footprint" "R_0805_2012Metric_Pad1.20x1.40mm_HandSolder"
 			(at 201.93 83.82 0)
 			(hide yes)
@@
 			)
 		)
-		(property "Footprint" "Vibra_Reviewed:TestPoint_Pad_D1.5mm"
+		(property "Footprint" "TestPoint_Pad_D1.5mm"
 			(at 68.58 153.67 0)
 			(hide yes)
@@
 			)
 		)
-		(property "Footprint" "Vibra_Reviewed:R_0805_2012Metric_Pad1.20x1.40mm_HandSolder"
+		(property "Footprint" "R_0805_2012Metric_Pad1.20x1.40mm_HandSolder"
 			(at 134.62 109.22 0)
 			(hide yes)
@@
 			)
 		)
-		(property "Footprint" "Vibra_Reviewed:TestPoint_Pad_D1.5mm"
+		(property "Footprint" "TestPoint_Pad_D1.5mm"
 			(at 25.4 153.67 0)
 			(hide yes)
@@
 			)
 		)
-		(property "Footprint" "Vibra_Reviewed:R_0805_2012Metric_Pad1.20x1.40mm_HandSolder"
+		(property "Footprint" "R_0805_2012Metric_Pad1.20x1.40mm_HandSolder"
 			(at 97.79 109.22 0)
 			(hide yes)
@@
 			)
 		)
-		(property "Footprint" "Vibra_Reviewed:TestPoint_Pad_D1.5mm"
+		(property "Footprint" "TestPoint_Pad_D1.5mm"
 			(at 198.12 153.67 0)
 			(hide yes)
@@
 			)
 		)
-		(property "Footprint" "Vibra_Reviewed:MountingHole_2.5mm"
+		(property "Footprint" "MountingHole_2.5mm"
 			(at 139.7 175.26 0)
 			(hide yes)
@@
 			)
 		)
-		(property "Footprint" "Vibra_Reviewed:R_0805_2012Metric_Pad1.20x1.40mm_HandSolder"
+		(property "Footprint" "R_0805_2012Metric_Pad1.20x1.40mm_HandSolder"
 			(at 38.1 80.01 0)
 			(hide yes)
@@
 			)
 		)
-		(property "Footprint" "Vibra_Reviewed:LED_0805_2012Metric_Pad1.15x1.40mm_HandSolder"
+		(property "Footprint" "LED_0805_2012Metric_Pad1.15x1.40mm_HandSolder"
 			(at 245.11 124.46 0)
 			(hide yes)
@@
 			)
 		)
-		(property "Footprint" "Vibra_Reviewed:C_0805_2012Metric_Pad1.18x1.45mm_HandSolder"
+		(property "Footprint" "C_0805_2012Metric_Pad1.18x1.45mm_HandSolder"
 			(at 269.24 68.58 0)
 			(hide yes)
@@
 			)
 		)
-		(property "Footprint" "Vibra_Reviewed:R_0805_2012Metric_Pad1.20x1.40mm_HandSolder"
+		(property "Footprint" "R_0805_2012Metric_Pad1.20x1.40mm_HandSolder"
 			(at 245.11 109.22 0)
 			(hide yes)
@@
 			)
 		)
-		(property "Footprint" "Vibra_Reviewed:TestPoint_Pad_D1.5mm"
+		(property "Footprint" "TestPoint_Pad_D1.5mm"
 			(at 241.3 153.67 0)
 			(hide yes)
@@
 			)
 		)
-		(property "Footprint" "Vibra_Reviewed:R_0805_2012Metric_Pad1.20x1.40mm_HandSolder"
+		(property "Footprint" "R_0805_2012Metric_Pad1.20x1.40mm_HandSolder"
 			(at 171.45 109.22 0)
 			(hide yes)
@@
 			)
 		)
-		(property "Footprint" "Vibra_Reviewed:LED_0805_2012Metric_Pad1.15x1.40mm_HandSolder"
+		(property "Footprint" "LED_0805_2012Metric_Pad1.15x1.40mm_HandSolder"
 			(at 134.62 124.46 0)
 			(hide yes)
@@
 			)
 		)
-		(property "Footprint" "Vibra_Reviewed:LED_0805_2012Metric_Pad1.15x1.40mm_HandSolder"
+		(property "Footprint" "LED_0805_2012Metric_Pad1.15x1.40mm_HandSolder"
 			(at 171.45 124.46 0)
 			(hide yes)
@@
 			)
 		)
-		(property "Footprint" "Vibra_Reviewed:R_0805_2012Metric_Pad1.20x1.40mm_HandSolder"
+		(property "Footprint" "R_0805_2012Metric_Pad1.20x1.40mm_HandSolder"
 			(at 208.28 109.22 0)
 			(hide yes)
@@
 			)
 		)
-		(property "Footprint" "Vibra_Reviewed:MountingHole_3.2mm_M3"
+		(property "Footprint" "MountingHole_3.2mm_M3"
 			(at 106.68 175.26 0)
 			(hide yes)
@@
 			)
 		)
-		(property "Footprint" "Vibra_Reviewed:LED_0805_2012Metric_Pad1.15x1.40mm_HandSolder"
+		(property "Footprint" "LED_0805_2012Metric_Pad1.15x1.40mm_HandSolder"
 			(at 97.79 124.46 0)
 			(hide yes)
